File: cad/SwiftSoilMoistureZigbeeSensor/SwiftSoilMoistureZigbeeSensor.kicad_sch (KiCad schematic)
At the start: 13 parts, among them J1 Probe, J3 ARM SWD, Q1 BSS84, SW1 Factory Reset, U1 TPS61221DCK, U2 E73-2G4M08S1C

Commit message: Replaced Jumper with SB
Parts:
- JP1: footprint Connector_PinHeader_2.54mm:PinHeader_1x02_P2.54mm_Vertical -> Jumper:SolderJumper-2_P1.3mm_Open_RoundedPad1.0x1.5mm; symbol Jumper:Jumper_2_Bridged -> Jumper:SolderJumper_2_Open
Changed lines of the file:
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@@
     (stroke (width 0) (type default))
   )
-  (wire (pts (xy 227.33 45.72) (xy 227.33 49.53))
-    (stroke (width 0) (type default))
-  )
-  (wire (pts (xy 227.33 33.02) (xy 227.33 35.56))
+  (wire (pts (xy 227.33 44.45) (xy 227.33 49.53))
+    (stroke (width 0) (type default))
+  )
+  (wire (pts (xy 227.33 33.02) (xy 227.33 36.83))
     (stroke (width 0) (type default))
   )
@@
     )
   )
-  (symbol (lib_id "Jumper:Jumper_2_Bridged") (at 227.33 40.64 90) (unit 1)
+  (symbol (lib_id "Jumper:SolderJumper_2_Open") (at 227.33 40.64 90) (unit 1)
     (in_bom yes) (on_board yes) (dnp no) (fields_autoplaced)
-    (property "Reference" "JP1" (at 228.6 39.37 90)
+    (property "Reference" "JP1" (at 229.87 39.37 90)
       (effects (font (size 1.27 1.27)) (justify right))
     )
-    (property "Value" "Jumper_Prog" (at 228.6 41.91 90)
+    (property "Value" "Jumper_Prog" (at 229.87 41.91 90)
       (effects (font (size 1.27 1.27)) (justify right))
     )
-    (property "Footprint" "Connector_PinHeader_2.54mm:PinHeader_1x02_P2.54mm_Vertical" (at 227.33 40.64 0)
-      (effects (font (size 1.27 1.27)) hide)
-    )
+    (property "Footprint" "Jumper:SolderJumper-2_P1.3mm_Open_RoundedPad1.0x1.5mm" (at 227.33 40.64 0)
+      (effects (font (size 1.27 1.27)) hide)
+    )

Commit message: Removed Jumper/SB
Parts:
- removed JP1: Jumper_Prog, Jumper:SolderJumper-2_P1.3mm_Open_RoundedPad1.0x1.5mm, symbol Jumper:SolderJumper_2_Open
Connections:
- net +3.3V: now also C2.1, Q1.2 (S), U1.2 (FB), U1.4 (VOUT)
Changed lines of the file:
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@@
   (title_block
     (title "Swift Zigbee Soil Moisture Sensor")
-    (date "2024-09-10")
-    (rev "1.2")
+    (date "2024-10-05")
+    (rev "1.3")
   )
   (junction (at 196.85 60.96) (diameter 0) (color 0 0 0 0)
@@
     (stroke (width 0) (type default))
   )
-  (wire (pts (xy 227.33 44.45) (xy 227.33 49.53))
-    (stroke (width 0) (type default))
-  )
-  (wire (pts (xy 227.33 33.02) (xy 227.33 36.83))
+  (wire (pts (xy 227.33 33.02) (xy 227.33 49.53))
     (stroke (width 0) (type default))
   )
@@
         )
       )
-    )
-  )
-  (symbol (lib_id "Jumper:SolderJumper_2_Open") (at 227.33 40.64 90) (unit 1)
-    (in_bom yes) (on_board yes) (dnp no) (fields_autoplaced)
-    (property "Reference" "JP1" (at 229.87 39.37 90)
-      (effects (font (size 1.27 1.27)) (justify right))
-    )
-    (property "Value" "Jumper_Prog" (at 229.87 41.91 90)
-      (effects (font (size 1.27 1.27)) (justify right))
-    )
-    (property "Footprint" "Jumper:SolderJumper-2_P1.3mm_Open_RoundedPad1.0x1.5mm" (at 227.33 40.64 0)
-      (effects (font (size 1.27 1.27)) hide)
-    )
-    (property "Datasheet" "~" (at 227.33 40.64 0)
-      (effects (font (size 1.27 1.27)) hide)
-    )
-    (property "LCSC" "C492401 + C3715628" (at 227.33 40.64 0)
-      (effects (font (size 1.27 1.27)) hide)
-    )
-    (pin "1")
-    (pin "2")
-    (instances
-      (project "SwiftSoilMoistureZigbeeSensor"
-        (path "/abcc6947-5804-4900-9240-6fa6b27c7542"
-          (reference "JP1") (unit 1)
-        )
-      )
